File: PCB/THD_Ver/nqgTHD.sch (KiCad schematic (older format))
At the start: 83 parts, among them J1 Conn_01x03, J2 Conn_01x03, J3 Conn_01x03, SW1 SW_PUSH, SW10 SW_PUSH, SW11 SW_PUSH, SW12 SW_PUSH, SW13 SW_PUSH, SW14 SW_PUSH, SW15 SW_PUSH, SW16 SW_PUSH, SW17 SW_PUSH, SW18 SW_PUSH, SW19 SW_PUSH, SW2 SW_PUSH, SW20 SW_PUSH, SW21 SW_PUSH, SW22 SW_PUSH, SW23 SW_PUSH, SW24 SW_PUSH, SW25 SW_PUSH, SW26 SW_PUSH, SW27 SW_PUSH, SW28 SW_PUSH, SW29 SW_PUSH, SW3 SW_PUSH, SW30 SW_PUSH, SW31 SW_PUSH, SW32 SW_PUSH, SW33 SW_PUSH, SW34 SW_PUSH, SW35 SW_PUSH, SW36 SW_PUSH, SW37 SW_PUSH, SW38 SW_PUSH, SW39 SW_PUSH, SW4 SW_PUSH, SW40 SW_PUSH, SW41 SW_PUSH, SW5 SW_PUSH, SW6 SW_PUSH, SW7 SW_PUSH, SW8 SW_PUSH, SW9 SW_PUSH, U1 ProMicro

Commit message: added THD version, removed beta_01
Parts:
- removed D38: D, Keebio-Parts:Diode-Hybrid-Back, symbol Device:D
- removed J1, J2, J3: Conn_01x03, emptystring:LEDStrip, symbol Connector_Generic:Conn_01x03
- removed SW20, SW25: SW_PUSH, emptystring:CherryMX_Hotswap_Back, symbol kbd:SW_PUSH
- removed SW41: SW_PUSH, kbd:ResetSW, symbol kbd:SW_PUSH
- added SW38, SW39: SW_PUSH, emptystring:CherryMX_Hotswap_Back, symbol kbd:SW_PUSH
- SW40: footprint emptystring:CherryMX_Hotswap_Back -> kbd:ResetSW
- U1: footprint emptystring:ProMicro_v2_Backside -> kbd:ProMicro_v2_Backside
- renumbered SW21 to SW20, SW22 to SW21, SW23 to SW22, SW24 to SW23, SW26 to SW24, SW27 to SW25, SW28 to SW26, SW29 to SW27, SW30 to SW28, SW31 to SW29, SW32 to SW30, SW33 to SW31, SW34 to SW32, SW35 to SW33, SW36 to SW34, SW37 to SW35, SW38 to SW36, SW39 to SW37
Connections:
- net labels removed: LED
- wire segments 95 -> 92
- no-connect marks 4 -> 5
