File: PCB/SMD_Ver/nqg.sch (KiCad schematic (older format))
At the start: 78 parts, among them SW1 SW_PUSH, SW10 SW_PUSH, SW11 SW_PUSH, SW12 SW_PUSH, SW13 SW_PUSH, SW14 SW_PUSH, SW15 SW_PUSH, SW16 SW_PUSH, SW17 SW_PUSH, SW18 SW_PUSH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

Commit message: added new screw to THD version, created new plates with new screw locations
Parts:
- U1: symbol kbd:ProMicro -> nqg-rescue:ProMicro-kbd
Changed lines of the file:
@@
 $EndDescr
 $Comp
-L kbd:ProMicro U1
+L nqg-rescue:ProMicro-kbd U1
 U 1 1 5C8B76EA
 P 13500 2300
